Commit message: calibration with controller for pi

File: description/camera.xacro (robot description, xacro)
@@ -4,10 +4,11 @@
         <parent link="chassis"/>
         <child link="camera_link"/>
-        <origin xyz="0.305 0 0.08" rpy="0 0 0"/>
+        <origin xyz="0.122495 0.122725 0.086129" rpy="0 0 0"/>
     </joint>
     <link name="camera_link">
         <visual>
+            <origin xyz="-0.122495 -0.122725 -0.086129" rpy="0 0 0"/>
             <geometry>
-                <box size="0.010 0.03 0.03"/>
+                <mesh filename="file://$(find ROS_rover_urdf_description)/meshes/Cam_1.stl" scale="0.001 0.001 0.001"/>
             </geometry>
             <material name="red"/>

File: description/gazebo_control.xacro (robot description, xacro)
@@ -6,6 +6,6 @@
             <left_joint>left_wheel_joint</left_joint>
             <right_joint>right_wheel_joint</right_joint>
-            <wheel_separation>0.35</wheel_separation>
-            <wheel_diameter>0.1</wheel_diameter>
+            <wheel_separation>0.1716</wheel_separation>
+            <wheel_diameter>0.078</wheel_diameter>
             <!-- Limits -->
             <max_wheel_torque>200</max_wheel_torque>

File: description/lidar.xacro (robot description, xacro)
@@ -4,21 +4,25 @@
         <parent link="chassis"/>
         <child link="laser_frame"/>
-        <origin xyz="0.1 0 0.175" rpy="0 0 0"/>
+        <origin xyz="-0.024813 0.122765 0.162152" rpy="0 0 0"/>
     </joint>
     <link name="laser_frame">
         <visual>
+            <origin xyz="0.024813 -0.122765 -0.162152" rpy="0 0 0"/>
             <geometry>
-                <cylinder radius="0.05" length="0.04"/>
+                <mesh filename="file://$(find ROS_rover_urdf_description)/meshes/Lidar_1.stl" scale="0.001 0.001 0.001"/>
             </geometry>
             <material name="red"/>
         </visual>
         <collision>
+            <origin xyz="0.024813 -0.122765 -0.162152" rpy="0 0 0"/>
             <geometry>
-                <cylinder radius="0.05" length="0.04"/>
+                <mesh filename="file://$(find ROS_rover_urdf_description)/meshes/Lidar_1.stl" scale="0.001 0.001 0.001"/>
             </geometry>
         </collision>
-        <xacro:inertial_cylinder mass="0.1" length="0.04" radius="0.05">
-            <origin xyz="0 0 0" rpy="0 0 0"/>
-        </xacro:inertial_cylinder>
+        <inertial>
+            <origin xyz="8.458430520580373e-08 -2.3180009273149338e-07 0.012473784183963443" rpy="0 0 0"/>
+            <mass value="0.5822410911588851"/>
+            <inertia ixx="0.000168" iyy="0.000168" izz="0.000275" ixy="0.0" iyz="0.0" ixz="0.0"/>
+        </inertial>
     </link>
     <gazebo reference="laser_frame">
@@ -26,5 +30,5 @@
         <sensor name="laser" type="ray">
             <pose> 0 0 0 0 0 0 </pose>
-            <visualize>false</visualize>
+            <visualize>true</visualize>
             <update_rate>10</update_rate>
             <ray>
@@ -43,5 +47,5 @@
             <plugin name="laser_controller" filename="libgazebo_ros_ray_sensor.so">
                 <ros>
-                    <argument>~/out:=scan</argument>
+                    <argument>--ros-args --remap ~/out:=scan</argument>
                 </ros>
                 <output_type>sensor_msgs/LaserScan</output_type>

File: description/robot.urdf.xacro (robot description, xacro)
@@ -1,8 +1,15 @@
 <?xml version="1.0"?>
 <robot xmlns:xacro="http://www.ros.org/wiki/xacro"  name="robot">
+    <xacro:arg name="use_ros2_control" default="true"/>
+    <xacro:arg name="sim_mode" default="false"/>
     <xacro:include filename="robot_core.xacro" />
-    <xacro:include filename="gazebo_control.xacro"/>
+    <xacro:if value="$(arg use_ros2_control)" >
+        <xacro:include filename="ros2_control.xacro"/>
+    </xacro:if>
+    <xacro:unless value="$(arg use_ros2_control)" >
+        <xacro:include filename="gazebo_control.xacro"/>
+    </xacro:unless>
     <xacro:include filename="lidar.xacro"/>
-    <!-- <xacro:include filename="camera.xacro"/> -->
-    <xacro:include filename="depth_camera.xacro"/>
+    <xacro:include filename="camera.xacro"/>
+    <!-- <xacro:include filename="depth_camera.xacro"/> -->
 </robot>

File: description/robot_core.xacro (robot description, xacro)
@@ -2,4 +2,7 @@
 <robot xmlns:xacro="http://www.ros.org/wiki/xacro"  >
     <xacro:include filename="inertial_macros.xacro"/>
+    <xacro:include filename="$(find ROS_rover_urdf_description)/urdf/materials.xacro" />
+    <xacro:include filename="$(find ROS_rover_urdf_description)/urdf/ROS_rover_urdf.trans" />
+    <xacro:include filename="$(find ROS_rover_urdf_description)/urdf/ROS_rover_urdf.gazebo" />
     <material name="white">
         <color rgba="1 1 1 1" />
@@ -19,4 +22,13 @@
 <!-- BASE LINK -->
     <link name="base_link">
+      <origin xyz="0 0 0" rpy="0 0 0"/>
+    </link>
+    <!-- BASE_FOOTPRINT LINK -->
+    <joint name="base_footprint_joint" type="fixed">
+        <parent link="base_link"/>
+        <child link="base_footprint"/>
+        <origin xyz="0 0 0" rpy="0 0 0"/>
+    </joint>
+    <link name="base_footprint">
     </link>
 <!-- CHASSIS LINK -->
@@ -24,23 +36,25 @@
         <parent link="base_link" />
         <child link="chassis" />
-        <origin xyz="-0.1 0 0"/>
+        <origin xyz="0.108526747687202506 -0.12224166560310168 -0.08643892236095495"/>
     </joint>
     <link name="chassis">
-        <visual>
-            <origin xyz="0.15 0 0.075"/>
+        <inertial>
+            <origin xyz="-0.018526747687202506 0.12224166560310168 0.08643892236095495" rpy="0 0 0"/>
+            <mass value="34.90606826800328"/>
+            <inertia ixx="0.114886" iyy="0.239343" izz="0.249193" ixy="0.000401" iyz="-0.000589" ixz="0.025841"/>
+          </inertial>
+          <visual>
+            <origin xyz="0 0 0" rpy="0 0 0"/>
             <geometry>
-                <box size="0.3 0.3 0.15" />
+              <mesh filename="file://$(find ROS_rover_urdf_description)/meshes/base_link.stl" scale="0.001 0.001 0.001"/>
             </geometry>
             <material name="white"/>
-        </visual>
-        <collision>
-            <origin xyz="0.15 0 0.075"/>
+          </visual>
+          <collision>
+            <origin xyz="0 0 0" rpy="0 0 0"/>
             <geometry>
-                <box size="0.3 0.3 0.15" />
+              <mesh filename="file://$(find ROS_rover_urdf_description)/meshes/base_link.stl" scale="0.001 0.001 0.001"/>
             </geometry>
-        </collision>
-        <xacro:inertial_box mass="0.5" x="0.3" y="0.3" z="0.15">
-            <origin xyz="0.15 0 0.075" rpy="0 0 0"/>
-        </xacro:inertial_box>
+          </collision>
     </link>
     <gazebo reference="chassis">
@@ -49,24 +63,28 @@
 <!-- LEFT WHEEL LINK-->
     <joint name="left_wheel_joint" type="continuous">
-        <parent link="base_link"/>
+        <parent link="chassis"/>
         <child link="left_wheel"/>
-        <origin xyz="0 0.175 0" rpy="-${pi/2} 0 0"/>
-        <axis xyz="0 0 1"/>
+        <origin xyz="-0.109883 0.2086 0.041686" rpy="0 0 0"/>
+        <axis xyz="0 1 0"/>
     </joint>
     <link name="left_wheel">
-        <visual>
+        <inertial>
+            <origin xyz="4.24215932839922e-07 0.01849999999999999 8.092045233193401e-08" rpy="0 0 0"/>
+            <mass value="1.3878753666636712"/>
+            <inertia ixx="0.000686" iyy="0.001055" izz="0.000686" ixy="0.0" iyz="0.0" ixz="-0.0"/>
+          </inertial>
+          <visual>
+            <origin xyz="0.109883 -0.2086 -0.041686" rpy="0 0 0"/>
             <geometry>
-                <cylinder radius="0.05" length="0.04"/>
+              <mesh filename="file://$(find ROS_rover_urdf_description)/meshes/Left_wheel_1.stl" scale="0.001 0.001 0.001"/>
             </geometry>
             <material name="blue"/>
-        </visual>
-        <collision>
+          </visual>
+          <collision>
+            <origin xyz="0.109883 -0.2086 -0.041686" rpy="0 0 0"/>
             <geometry>
-                <cylinder radius="0.05" length="0.04"/>
+              <mesh filename="file://$(find ROS_rover_urdf_description)/meshes/Left_wheel_1.stl" scale="0.001 0.001 0.001"/>
             </geometry>
-        </collision>
-        <xacro:inertial_cylinder mass="0.1" length="0.04" radius="0.05">
-            <origin xyz="0 0 0" rpy="0 0 0"/>
-        </xacro:inertial_cylinder>
+          </collision>
     </link>
     <gazebo reference="left_wheel">
@@ -75,24 +93,28 @@
 <!-- RIGHT WHEEL LINK-->
 <joint name="right_wheel_joint" type="continuous">
-    <parent link="base_link"/>
+    <origin xyz="-0.109883 0.037 0.041686" rpy="0 0 0"/>
+    <parent link="chassis"/>
     <child link="right_wheel"/>
-    <origin xyz="0 -0.175 0" rpy="${pi/2} 0 0"/>
-    <axis xyz="0 0 -1"/>
+    <axis xyz="0.0 1.0 0.0"/>
 </joint>
 <link name="right_wheel">
-    <visual>
+    <inertial>
+        <origin xyz="4.24215932839922e-07 -0.018500000000000003 8.09204523458118e-08" rpy="0 0 0"/>
+        <mass value="1.3878753666636718"/>
+        <inertia ixx="0.000686" iyy="0.001055" izz="0.000686" ixy="-0.0" iyz="0.0" ixz="-0.0"/>
+      </inertial>
+      <visual>
+        <origin xyz="0.109883 -0.037 -0.041686" rpy="0 0 0"/>
         <geometry>
-            <cylinder radius="0.05" length="0.04"/>
+          <mesh filename="file://$(find ROS_rover_urdf_description)/meshes/Right_wheel_1.stl" scale="0.001 0.001 0.001"/>
         </geometry>
         <material name="blue"/>
-    </visual>
-    <collision>
+      </visual>
+      <collision>
+        <origin xyz="0.109883 -0.037 -0.041686" rpy="0 0 0"/>
         <geometry>
-            <cylinder radius="0.05" length="0.04"/>
+          <mesh filename="file://$(find ROS_rover_urdf_description)/meshes/Right_wheel_1.stl" scale="0.001 0.001 0.001"/>
         </geometry>
-    </collision>
-    <xacro:inertial_cylinder mass="0.1" length="0.04" radius="0.05">
-            <origin xyz="0 0 0" rpy="0 0 0"/>
-    </xacro:inertial_cylinder>
+      </collision>
 </link>
 <gazebo reference="right_wheel">
@@ -103,21 +125,26 @@
     <parent link="chassis"/>
     <child link="castor_wheel"/>
-    <origin xyz="0.24 0 0"/>
+    <origin xyz="0.05652 0.121748 0.027021" rpy="0 0 0"/>
+    <axis xyz="0.0 0.0 -1.0"/>
 </joint>
 <link name="castor_wheel">
-    <visual>
+    <inertial>
+        <origin xyz="2.7755575615628914e-17 -1.4670485243284404e-08 3.1211140116491065e-07" rpy="0 0 0"/>
+        <mass value="0.4809809344697313"/>
+        <inertia ixx="0.000115" iyy="0.000115" izz="0.000115" ixy="0.0" iyz="0.0" ixz="0.0"/>
+      </inertial>
+      <visual>
+        <origin xyz="-0.05652 -0.121748 -0.027021" rpy="0 0 0"/>
         <geometry>
-            <sphere radius="0.05" />
+          <mesh filename="file://$(find ROS_rover_urdf_description)/meshes/_front_ball_1.stl" scale="0.001 0.001 0.001"/>
         </geometry>
         <material name="black"/>
-    </visual>
-    <collision>
+      </visual>
+      <collision>
+        <origin xyz="-0.05652 -0.121748 -0.027021" rpy="0 0 0"/>
         <geometry>
-            <sphere radius="0.05" />
+          <mesh filename="file://$(find ROS_rover_urdf_description)/meshes/_front_ball_1.stl" scale="0.001 0.001 0.001"/>
         </geometry>
-    </collision>
-    <xacro:inertial_sphere mass="0.1" radius="0.05">
-        <origin xyz="0 0 0" rpy="0 0 0"/>
-    </xacro:inertial_sphere>
+      </collision>
 </link>
 <gazebo reference="castor_wheel">
